File: mp3/mp3.kicad_sch (KiCad schematic)
At the start: 33 parts, among them J1 USB4105-GF-A, J2 LEFT, J3 DEBUG, J4 RIGHT, U1 W25Q128JV, U2 RP2040, U3 MCP1702T-3302E_CB, Y1 12MHz

Commit message: Update new layout design according to Brad
Parts:
- C12: footprint Capacitor_SMD:C_0402_1005Metric -> Capacitor_SMD:C_0603_1608Metric
- C13: footprint Capacitor_SMD:C_0402_1005Metric -> Capacitor_SMD:C_0201_0603Metric
Changed lines of the file:
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@@
       (effects (font (size 1.27 1.27)) (justify right))
     )
-    (property "Footprint" "Capacitor_SMD:C_0402_1005Metric" (id 2) (at 178.7652 25.4 0)
+    (property "Footprint" "Capacitor_SMD:C_0603_1608Metric" (id 2) (at 178.7652 25.4 0)
       (effects (font (size 1.27 1.27)) hide)
     )
@@
       (effects (font (size 1.27 1.27)) (justify left))
     )
-    (property "Footprint" "Capacitor_SMD:C_0402_1005Metric" (id 2) (at 209.2452 33.02 0)
+    (property "Footprint" "Capacitor_SMD:C_0201_0603Metric" (id 2) (at 209.2452 33.02 0)
       (effects (font (size 1.27 1.27)) hide)
     )
@@
     )
     (path "/72143c83-9810-4c68-bdb6-6021f1d73d44"
-      (reference "C12") (unit 1) (value "10µF") (footprint "Capacitor_SMD:C_0402_1005Metric")
+      (reference "C12") (unit 1) (value "10µF") (footprint "Capacitor_SMD:C_0603_1608Metric")
     )
     (path "/7896dfda-1d9c-4d04-8928-a34570745fb1"
-      (reference "C13") (unit 1) (value "10µF") (footprint "Capacitor_SMD:C_0402_1005Metric")
+      (reference "C13") (unit 1) (value "10µF") (footprint "Capacitor_SMD:C_0201_0603Metric")
     )
     (path "/a4361543-0cee-4944-9d11-d5d7399a6613"

Commit message: Make changes on layout according to Brad
Parts:
- C1: footprint Resistor_SMD:R_0201_0603Metric -> Resistor_SMD:R_0402_1005Metric
- C13: footprint Capacitor_SMD:C_0201_0603Metric -> Capacitor_SMD:C_0603_1608Metric
Changed lines of the file:
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@@
       (effects (font (size 1.27 1.27)) (justify right))
     )
-    (property "Footprint" "Resistor_SMD:R_0201_0603Metric" (id 2) (at 25.0952 96.52 0)
+    (property "Footprint" "Resistor_SMD:R_0402_1005Metric" (id 2) (at 25.0952 96.52 0)
       (effects (font (size 1.27 1.27)) hide)
     )
@@
       (effects (font (size 1.27 1.27)) (justify left))
     )
-    (property "Footprint" "Capacitor_SMD:C_0201_0603Metric" (id 2) (at 209.2452 33.02 0)
+    (property "Footprint" "Capacitor_SMD:C_0603_1608Metric" (id 2) (at 209.2452 33.02 0)
       (effects (font (size 1.27 1.27)) hide)
     )
@@
     )
     (path "/2fc9b624-be90-48f2-b80c-7987b933913b"
-      (reference "C1") (unit 1) (value "0.1µF") (footprint "Resistor_SMD:R_0201_0603Metric")
+      (reference "C1") (unit 1) (value "0.1µF") (footprint "Resistor_SMD:R_0402_1005Metric")
     )
     (path "/e23992fa-79b5-4597-9d36-5463246aaeb4"
@@
     )
     (path "/7896dfda-1d9c-4d04-8928-a34570745fb1"
-      (reference "C13") (unit 1) (value "10µF") (footprint "Capacitor_SMD:C_0201_0603Metric")
+      (reference "C13") (unit 1) (value "10µF") (footprint "Capacitor_SMD:C_0603_1608Metric")
     )
     (path "/a4361543-0cee-4944-9d11-d5d7399a6613"
